File: hardware/main-controller/kicad/agrinode_mc.kicad_pcb (KiCad board)
At the start: 4 copper layers, 240 x 180 mm, 319 parts, among them J1 MAIN IN 9-32V, J10 RELAY 2, J11 RELAY 3, J12 RELAY 4, J13 RELAY 5, J14 RELAY 6, J15 RELAY 7, J16 RELAY 8, J17 DI 1-4, J18 DI 5-8, J19 AI 1-2, J2 BATTERY IN 9-32V, J20 AI 3-4, J21 AO 1-2, J22 OUT 1-2, J23 OUT 3-4, J24 1-WIRE, J25 I2C EXT, J26 RS485-A EXP BUS, J27 RS485-B FIELD, J3 USB-C, J4 SPARE IO, J5 OLED I2C, J6 ETHERNET, J7 microSD, J8 MODEM SLOT, J9 RELAY 1, K1 SRD-05VDC-SL-C, K2 SRD-05VDC-SL-C, K3 SRD-05VDC-SL-C, K4 SRD-05VDC-SL-C, K5 SRD-05VDC-SL-C, K6 SRD-05VDC-SL-C, K7 SRD-05VDC-SL-C, K8 SRD-05VDC-SL-C, Q1 MMBT3904, Q2 IRLR2905, Q3 IRLR2905, Q4 IRLR2905, Q5 IRLR2905, SW1 RESET, SW2 BOOT / OK, SW3 UP, SW4 DOWN, SW5 BACK, U1 TPS54360DDA, U10 Ra-02 SX1278 433MHz, U11 PCA9555D, U12 ULN2803A, U13 TLP290-4, U14 TLP290-4, U15 ADS1115IDGS, U16 MCP4728, U17 OPA2196xD, U18 74AHCT1G125, U19 74AHCT1G125, U2 TPS563200, U20 74AHCT1G125, U21 74AHCT1G125, U22 USBLC6-2SC6, U23 THVD1420D, U24 ADM2587E, U3 ESP32-S3-WROOM-1-N16R2, U4 USBLC6-2SC6, U5 TPL5010, U6 DS3231MZ, U7 ATECC608B-TNGTLS (I2C 0x35), U8 PCA9555D, U9 W5500, Y1 25MHz 18pF

Commit message: Route MC-1 PCB with Freerouting and import the session
- 3083 track segments, 626 vias; 0 clearance violations, 48 connections
  left for manual completion (mostly plane hookups)
- relay contact tracks (10 A / 250 VAC) moved to both outer layers
- DRC now runs after net classes are re-resolved from the project file
- VBUS_USB uses the fine-pitch class so the USB-C pads pass clearance

Co-Authored-By: Claude Opus 5.5 <noreply@anthropic.com>
Claude-Session: https://claude.ai/code/session_014J7amXZ5Y6AZWEh5CjDNja
Routing:
- net +5V: track 0.00 -> 746.0 mm, vias 0 -> 4
- net I2C_SDA: track 0.00 -> 631.8 mm, vias 0 -> 9
- net I2C_SCL: track 0.00 -> 447.3 mm, vias 0 -> 12
- net GND: track 0.00 -> 430.8 mm, vias 0 -> 182
- net VFIELD: track 0.00 -> 350.7 mm, vias 0 -> 6
- net RS485B_DE: track 0.00 -> 308.8 mm, vias 0 -> 3
- net DI1: track 0.00 -> 269.2 mm, vias 0 -> 5
- net DI2: track 0.00 -> 259.6 mm, vias 0 -> 3
- net RS485B_RX: track 0.00 -> 244.0 mm, vias 0 -> 5
- net RS485A_DE: track 0.00 -> 241.9 mm, vias 0 -> 3
- net RS485B_TX: track 0.00 -> 234.2 mm, vias 0 -> 5
- net RS485A_RX: track 0.00 -> 233.9 mm, vias 0 -> 5
- net VIN_MAIN_SENSE: track 0.00 -> 229.4 mm, vias 0 -> 4
- net RS485A_TX: track 0.00 -> 226.7 mm, vias 0 -> 3
- net VIN_BAT_SENSE: track 0.00 -> 221.1 mm, vias 0 -> 2
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- added copper zone on B.Cu, net GND
- added copper zone on F.Cu, net GND
- added copper zone on B.Cu, net GND_ISO
- added copper zone on F.Cu, net GND_ISO
