File: hardware/hubs/hub-c/kicad/mcu.kicad_sch (KiCad schematic)
At the start: 38 parts, among them J6 PROG, J7 I2C, J8 LED STRIP WS2813, Q3 MMBT3904, Q4 MMBT3904, Q5 BSS138, Q6 MMBT3904, SW1 RESET, SW2 BOOT / PAIR, U4 ESP32-WROOM-32E-N8, U5 CH340C, U6 DS3231MZ

Commit message: hubs: remap ESP32 GPIOs to the module side facing each block; keep-best rip-up stages
RS-485 moves to IO17/16/4 (right column, next to the RS-485 block), I2C to
IO33/32, charger status to IO13 (bottom row, no strapping pin), LoRa DIO0/RST
and the LTE control lines to right-column pins. Rip-up stages now keep a
result only when it leaves fewer open nets.

Co-Authored-By: Claude Opus 5.5 <noreply@anthropic.com>
Claude-Session: https://claude.ai/code/session_014J7amXZ5Y6AZWEh5CjDNja
Connections:
- net CHRG_N: now also U4.16 (IO13); no longer U4.14 (IO12)
- net I2C_SCL: now also U4.8 (IO32); no longer U4.36 (IO22)
- net I2C_SDA: now also U4.9 (IO33); no longer U4.33 (IO21)
- net MODEM_EN: now also U4.36 (IO22); no longer U4.23 (IO15)
- net MODEM_PWRKEY_CTL: now also U4.33 (IO21); no longer U4.16 (IO13)
- net MODEM_RXD: now also U4.31 (IO19); no longer U4.27 (IO16)
- net MODEM_STATUS: now also U4.30 (IO18); no longer U4.5 (SENSOR_VN)
- net MODEM_TXD: now also U4.37 (IO23); no longer U4.28 (IO17)
- net RS485_DE: now also U4.26 (IO4); no longer U4.10 (IO25)
- net RS485_RX: now also U4.27 (IO16); no longer U4.9 (IO33)
- net RS485_TX: now also U4.28 (IO17); no longer U4.8 (IO32)
Other:
- moved on the sheet: BT2, C14, C15, C16, C17, C18, C19, J6, J7, Q3, Q4, R13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
