File: hardware/hubs/hub-l/kicad/mcu.kicad_sch (KiCad schematic)
At the start: 38 parts, among them J6 PROG, J7 I2C, J8 LED STRIP WS2813, Q3 MMBT3904, Q4 MMBT3904, Q5 BSS138, Q6 MMBT3904, SW1 RESET, SW2 BOOT / PAIR, U4 ESP32-WROOM-32E-N8, U5 CH340C, U6 DS3231MZ

Commit message: hubs: remap ESP32 GPIOs to the module side facing each block; keep-best rip-up stages
RS-485 moves to IO17/16/4 (right column, next to the RS-485 block), I2C to
IO33/32, charger status to IO13 (bottom row, no strapping pin), LoRa DIO0/RST
and the LTE control lines to right-column pins. Rip-up stages now keep a
result only when it leaves fewer open nets.

Co-Authored-By: Claude Opus 5.5 <noreply@anthropic.com>
Claude-Session: https://claude.ai/code/session_014J7amXZ5Y6AZWEh5CjDNja
Connections:
- net CHRG_N: now also U4.16 (IO13); no longer U4.14 (IO12)
- net I2C_SCL: now also U4.8 (IO32); no longer U4.36 (IO22)
- net I2C_SDA: now also U4.9 (IO33); no longer U4.33 (IO21)
- net LORA_DIO0: now also U4.33 (IO21); no longer U4.11 (IO26)
- net LORA_RST: now also U4.36 (IO22); no longer U4.13 (IO14)
- net RS485_DE: now also U4.26 (IO4); no longer U4.10 (IO25)
- net RS485_RX: now also U4.27 (IO16); no longer U4.9 (IO33)
- net RS485_TX: now also U4.28 (IO17); no longer U4.8 (IO32)
Changed lines of the file:
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@@
     )
   )
-  (wire
-    (pts
-      (xy 58.42 81.28)
-      (xy 60.96 81.28)
-    )
-    (stroke
-      (width 0)
-      (type default)
-    )
-  )
-  (global_label "RS485_DE"
-    (shape passive)
-    (at 60.96 81.28 0)
-    (fields_autoplaced)
-    (effects
-      (font
-        (size 1.27 1.27)
-      )
-      (justify left)
-    )
-    (property "Intersheetrefs" "${INTERSHEET_REFS}"
-      (at 60.96 81.28 0)
-      (effects
-        (font
-          (size 1.27 1.27)
-        )
-        (justify left)
-        hide
-      )
-    )
-  )
-  (wire
-    (pts
-      (xy 58.42 83.82)
-      (xy 60.96 83.82)
-    )
-    (stroke
-      (width 0)
-      (type default)
-    )
-  )
-  (global_label "LORA_DIO0"
-    (shape passive)
-    (at 60.96 83.82 0)
-    (fields_autoplaced)
-    (effects
-      (font
-        (size 1.27 1.27)
-      )
-      (justify left)
-    )
-    (property "Intersheetrefs" "${INTERSHEET_REFS}"
-      (at 60.96 83.82 0)
-      (effects
-        (font
-          (size 1.27 1.27)
-        )
-        (justify left)
-        hide
-      )
-    )
+  (no_connect
+    (at 58.42 81.28)
+  )
+  (no_connect
+    (at 58.42 83.82)
   )
   (wire
@@
     )
   )
-  (wire
-    (pts
-      (xy 58.42 58.42)
-      (xy 60.96 58.42)
-    )
-    (stroke
-      (width 0)
-      (type default)
-    )
-  )
-  (global_label "LORA_RST"
-    (shape passive)
-    (at 60.96 58.42 0)
-    (fields_autoplaced)
-    (effects
-      (font
-        (size 1.27 1.27)
-      )
-      (justify left)
-    )
-    (property "Intersheetrefs" "${INTERSHEET_REFS}"
-      (at 60.96 58.42 0)
-      (effects
-        (font
-          (size 1.27 1.27)
-        )
-        (justify left)
-        hide
-      )
-    )
-  )
-  (wire
-    (pts
-      (xy 58.42 53.34)
-      (xy 60.96 53.34)
+  (no_connect
+    (at 58.42 58.42)
+  )
+  (no_connect
+    (at 58.42 53.34)
+  )
+  (wire
+    (pts
+      (xy 58.42 55.88)
+      (xy 60.96 55.88)
     )
     (stroke
@@
   (global_label "CHRG_N"
     (shape passive)
-    (at 60.96 53.34 0)
-    (fields_autoplaced)
-    (effects
-      (font
-        (size 1.27 1.27)
-      )
-      (justify left)
-    )
-    (property "Intersheetrefs" "${INTERSHEET_REFS}"
-      (at 60.96 53.34 0)
-      (effects
-        (font
-          (size 1.27 1.27)
-        )
-        (justify left)
-        hide
-      )
-    )
-  )
-  (no_connect
-    (at 58.42 55.88)
+    (at 60.96 55.88 0)
+    (fields_autoplaced)
+    (effects
+      (font
+        (size 1.27 1.27)
+      )
+      (justify left)
+    )
+    (property "Intersheetrefs" "${INTERSHEET_REFS}"
+      (at 60.96 55.88 0)
+      (effects
+        (font
+          (size 1.27 1.27)
+        )
+        (justify left)
+        hide
+      )
+    )
   )
   (no_connect
@@
     )
   )
-  (no_connect
-    (at 58.42 48.26)
-  )
-  (no_connect
-    (at 58.42 63.5)
-  )
-  (no_connect
-    (at 58.42 66.04)
+  (wire
+    (pts
+      (xy 58.42 48.26)
+      (xy 60.96 48.26)
+    )
+    (stroke
+      (width 0)
+      (type default)
+    )
+  )
+  (global_label "RS485_DE"
+    (shape passive)
+    (at 60.96 48.26 0)
+    (fields_autoplaced)
+    (effects
+      (font
+        (size 1.27 1.27)
+      )
+      (justify left)
+    )
+    (property "Intersheetrefs" "${INTERSHEET_REFS}"
+      (at 60.96 48.26 0)
+      (effects
+        (font
+          (size 1.27 1.27)
+        )
+        (justify left)
+        hide
+      )
+    )
+  )
+  (wire
+    (pts
+      (xy 58.42 63.5)
+      (xy 60.96 63.5)
+    )
+    (stroke
+      (width 0)
+      (type default)
+    )
+  )
+  (global_label "RS485_RX"
+    (shape passive)
+    (at 60.96 63.5 0)
+    (fields_autoplaced)
+    (effects
+      (font
+        (size 1.27 1.27)
+      )
+      (justify left)
+    )
+    (property "Intersheetrefs" "${INTERSHEET_REFS}"
+      (at 60.96 63.5 0)
+      (effects
+        (font
+          (size 1.27 1.27)
+        )
+        (justify left)
+        hide
+      )
+    )
+  )
+  (wire
+    (pts
+      (xy 58.42 66.04)
+      (xy 60.96 66.04)
+    )
+    (stroke
+      (width 0)
+      (type default)
+    )
+  )
+  (global_label "RS485_TX"
+    (shape passive)
+    (at 60.96 66.04 0)
+    (fields_autoplaced)
+    (effects
+      (font
+        (size 1.27 1.27)
+      )
+      (justify left)
+    )
+    (property "Intersheetrefs" "${INTERSHEET_REFS}"
+      (at 60.96 66.04 0)
+      (effects
+        (font
+          (size 1.27 1.27)
+        )
+        (justify left)
+        hide
+      )
+    )
   )
   (wire
@@
     )
   )
-  (label "I2C_SDA"
+  (global_label "LORA_DIO0"
+    (shape passive)
     (at 60.96 73.66 0)
     (fields_autoplaced)
@@
         (size 1.27 1.27)
       )
-      (justify left bottom)
+      (justify left)
+    )
+    (property "Intersheetrefs" "${INTERSHEET_REFS}"
+      (at 60.96 73.66 0)
+      (effects
+        (font
+          (size 1.27 1.27)
+        )
+        (justify left)
+        hide
+      )
     )
   )
@@
     )
   )
-  (label "I2C_SCL"
+  (global_label "LORA_RST"
+    (shape passive)
     (at 60.96 76.2 0)
     (fields_autoplaced)
@@
         (size 1.27 1.27)
       )
-      (justify left bottom)
+      (justify left)
+    )
+    (property "Intersheetrefs" "${INTERSHEET_REFS}"
+      (at 60.96 76.2 0)
+      (effects
+        (font
+          (size 1.27 1.27)
+        )
+        (justify left)
+        hide
+      )
     )
   )
@@
     )
   )
-  (global_label "RS485_TX"
-    (shape passive)
+  (label "I2C_SCL"
     (at 60.96 88.9 0)
     (fields_autoplaced)
@@
         (size 1.27 1.27)
       )
-      (justify left)
-    )
-    (property "Intersheetrefs" "${INTERSHEET_REFS}"
-      (at 60.96 88.9 0)
-      (effects
-        (font
-          (size 1.27 1.27)
-        )
-        (justify left)
-        hide
-      )
+      (justify left bottom)
     )
   )
@@
     )
   )
-  (global_label "RS485_RX"
-    (shape passive)
+  (label "I2C_SDA"
     (at 60.96 91.44 0)
     (fields_autoplaced)
@@
         (size 1.27 1.27)
       )
-      (justify left)
-    )
-    (property "Intersheetrefs" "${INTERSHEET_REFS}"
-      (at 60.96 91.44 0)
-      (effects
-        (font
-          (size 1.27 1.27)
-        )
-        (justify left)
-        hide
-      )
-    )
-  )
+      (justify left bottom)
+    )
+  )
