File: hardware/hubs/hub-l/kicad/agrinode_hub_l.kicad_pcb (KiCad board)
At the start: 2 copper layers, 130 x 96 mm, 105 parts, among them J1 DC 12V 5.5/2.1, J2 DC IN 7-24V, J3 SOLAR 6-24V, J4 USB 5V / PROG, J5 BAT NTC 10k, J6 PROG, J7 I2C, J8 LED STRIP WS2813, J9 RS-485, Q1 AO3401A, Q2 AO3401A, Q3 MMBT3904, Q4 MMBT3904, Q5 BSS138, Q6 MMBT3904, SW1 RESET, SW2 BOOT / PAIR, U1 LM2596S-5.0, U2 TP4056, U3 MIC29302WU, U4 ESP32-WROOM-32E-N8, U5 CH340C, U6 DS3231MZ, U7 MAX3485ESA, U8 Ra-02 SX1278 433MHz

Commit message: hubs: routing progress snapshot (HUB-L 3 open)
Co-Authored-By: Claude Opus 5.5 <noreply@anthropic.com>
Claude-Session: https://claude.ai/code/session_014J7amXZ5Y6AZWEh5CjDNja
Routing:
- net GND: track 0.00 -> 884.8 mm, vias 0 -> 8
- net +3V3: track 0.00 -> 399.1 mm, vias 0 -> 11
- net SPI_MOSI: track 0.00 -> 223.6 mm, vias 0 -> 8
- net /Power - 12V, solar and USB inputs, 18650 charger, rails/VUSB_RAW: track 0.00 -> 185.4 mm, vias 0 -> 1
- net /Power - 12V, solar and USB inputs, 18650 charger, rails/V5: track 0.00 -> 177.7 mm, vias 0 -> 2
- net VSYS: track 0.00 -> 177.2 mm, vias 0 -> 4
- net /ESP32, programming, buttons, RTC, LED strip, buzzer/ESP_TXD0: track 0.00 -> 132.4 mm, vias 0 -> 4
- net /ESP32, programming, buttons, RTC, LED strip, buzzer/BOOT_BTN: track 0.00 -> 96.7 mm, vias 0 -> 2
- net LORA_DIO0: track 0.00 -> 95.4 mm, vias 0 -> 4
- net /ESP32, programming, buttons, RTC, LED strip, buzzer/I2C_SCL: track 0.00 -> 92.5 mm, vias 0 -> 2
- net /ESP32, programming, buttons, RTC, LED strip, buzzer/I2C_SDA: track 0.00 -> 91.0 mm, vias 0 -> 1
- net /Power - 12V, solar and USB inputs, 18650 charger, rails/BATT_CELL: track 0.00 -> 89.4 mm, vias 0 -> 2
- net RS485_DE: track 0.00 -> 88.7 mm, vias 0 -> 2
- net /Power - 12V, solar and USB inputs, 18650 charger, rails/VBAT: track 0.00 -> 79.6 mm, vias 0 -> 3
- net LORA_CS: track 0.00 -> 79.1 mm, vias 0 -> 2
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- added copper zone on B.Cu, net GND
- added copper zone on F.Cu, net GND

Commit message: hubs: routing progress snapshot
Co-Authored-By: Claude Opus 5.5 <noreply@anthropic.com>
Claude-Session: https://claude.ai/code/session_014J7amXZ5Y6AZWEh5CjDNja
Parts:
- moved R26 34.2 mm to (156.5, 101.6)
- moved R27 28.3 mm to (162.4, 95.6)
- moved R7 28.1 mm to (145.7, 67.6)
- moved R8 28.1 mm to (145.7, 72.1)
- moved U6 17.5 mm to (137.7, 95.7), turned to 180 degrees
- moved JP2 17.0 mm to (142.9, 111.1)
- moved C21 15.7 mm to (144.2, 106.7)
- moved R31 13.4 mm to (162.7, 114.1)
- moved U7 11.0 mm to (157.9, 107.9)
- moved D10 9.98 mm to (162.7, 100.9)
- moved R28 9.08 mm to (136.3, 111.1)
- moved D9 8.29 mm to (152.5, 69.2)
- moved R22 6.20 mm to (137.6, 106.6)
- moved R21 4.50 mm to (137.6, 102.1)
- moved C10 2.73 mm to (146.2, 98.8)
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Routing:
- net GND: track 884.8 -> 0.00 mm, vias 8 -> 0
- net +3V3: track 399.1 -> 0.00 mm, vias 11 -> 0
- net SPI_MOSI: track 223.6 -> 0.00 mm, vias 8 -> 0
- net /Power - 12V, solar and USB inputs, 18650 charger, rails/VUSB_RAW: track 185.4 -> 0.00 mm, vias 1 -> 0
- net /Power - 12V, solar and USB inputs, 18650 charger, rails/V5: track 177.7 -> 0.00 mm, vias 2 -> 0
- net VSYS: track 177.2 -> 0.00 mm, vias 4 -> 0
- net /ESP32, programming, buttons, RTC, LED strip, buzzer/ESP_TXD0: track 132.4 -> 0.00 mm, vias 4 -> 0
- net /ESP32, programming, buttons, RTC, LED strip, buzzer/BOOT_BTN: track 96.7 -> 0.00 mm, vias 2 -> 0
- net LORA_DIO0: track 95.4 -> 0.00 mm, vias 4 -> 0
- net /ESP32, programming, buttons, RTC, LED strip, buzzer/I2C_SCL: track 92.5 -> 0.00 mm, vias 2 -> 0
- net /ESP32, programming, buttons, RTC, LED strip, buzzer/I2C_SDA: track 91.0 -> 0.00 mm, vias 1 -> 0
- net /Power - 12V, solar and USB inputs, 18650 charger, rails/BATT_CELL: track 89.4 -> 0.00 mm, vias 2 -> 0
- net RS485_DE: track 88.7 -> 0.00 mm, vias 2 -> 0
- net /Power - 12V, solar and USB inputs, 18650 charger, rails/VBAT: track 79.6 -> 0.00 mm, vias 3 -> 0
- net LORA_CS: track 79.1 -> 0.00 mm, vias 2 -> 0
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- removed copper zone on B.Cu, net GND
- removed copper zone on F.Cu, net GND
