File: hardware/hubs/gw-lan/kicad/agrinode_gw_lan.kicad_pcb (KiCad board)
At the start: 2 copper layers, 150 x 96 mm, 126 parts, among them J1 DC 12V 5.5/2.1, J10 LAN, J2 DC IN 7-24V, J3 SOLAR 6-24V, J4 USB 5V / PROG, J5 BAT NTC 10k, J6 PROG, J7 I2C, J8 LED STRIP WS2813, J9 RS-485, Q1 AO3401A, Q2 AO3401A, Q3 MMBT3904, Q4 MMBT3904, Q5 BSS138, Q6 MMBT3904, SW1 RESET, SW2 BOOT / PAIR, U1 LM2596S-5.0, U2 TP4056, U3 MIC29302WU, U4 ESP32-WROOM-32E-N8, U5 CH340C, U6 DS3231MZ, U7 MAX3485ESA, U8 Ra-02 SX1278 433MHz, U9 ENC28J60-I/SO, Y1 25MHz

Commit message: hubs: open a 6 mm routing channel beside the ESP32 right column (BOOT button and PROG header moved); pin the LDO bulk cap
Co-Authored-By: Claude Opus 5.5 <noreply@anthropic.com>
Claude-Session: https://claude.ai/code/session_014J7amXZ5Y6AZWEh5CjDNja
Parts:
- moved C10 131.6 mm to (106.2, 77.8)
- moved D7 42.6 mm to (57.6, 96.3)
- moved D8 40.9 mm to (127.1, 116.8)
- moved R8 25.6 mm to (141.8, 60.1)
- moved R2 24.5 mm to (113.3, 118.1)
- moved R3 23.8 mm to (106.3, 91.1)
- moved C9 23.7 mm to (135.0, 80.7)
- moved R21 23.6 mm to (127.9, 111.6)
- moved C11 21.9 mm to (136.4, 85.2)
- moved R6 21.6 mm to (136.4, 89.6)
- moved R18 21.1 mm to (153.5, 58.6)
- moved C7 18.2 mm to (102.4, 96.2)
- moved R22 17.9 mm to (143.1, 85.1)
- moved Q3 16.9 mm to (141.4, 54.9)
- moved C16 14.0 mm to (92.3, 78.2)
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