File: hardware/hubs/hub-w/kicad/agrinode_hub_w.kicad_pcb (KiCad board)
At the start: 2 copper layers, 114 x 96 mm, 101 parts, among them J1 DC 12V 5.5/2.1, J2 DC IN 7-24V, J3 SOLAR 6-24V, J4 USB 5V / PROG, J5 BAT NTC 10k, J6 PROG, J7 I2C, J8 LED STRIP WS2813, J9 RS-485, Q1 AO3401A, Q2 AO3401A, Q3 MMBT3904, Q4 MMBT3904, Q5 BSS138, Q6 MMBT3904, SW1 RESET, SW2 BOOT / PAIR, U1 LM2596S-5.0, U2 TP4056, U3 MIC29302WU, U4 ESP32-WROOM-32E-N8, U5 CH340C, U6 DS3231MZ, U7 MAX3485ESA

Commit message: hubs: GND stitching vias + GND left to the pours (autorouter routes signals only)
Co-Authored-By: Claude Opus 5.5 <noreply@anthropic.com>
Claude-Session: https://claude.ai/code/session_014J7amXZ5Y6AZWEh5CjDNja
Routing:
- net GND: track 0.00 -> 83.3 mm, vias 0 -> 62
